File: LED_Dimmer.brd (EAGLE design)
At the start: 48.3 x 62.2 mm, 12 parts

Commit message: Swapped Fet Drain and Source
Connections:
- removed net N$5: FETR.3, JP1.3, JP1.4
- new net N$7: FETR.2, JP1.3, JP1.4
- net GND: now also FETB.3, FETG.3, FETR.3; no longer FETB.2, FETG.2, FETR.2
- net N$4: now also FETB.2; no longer FETB.3
- net N$6: now also FETG.2; no longer FETG.3
Routing:
- net N$5: track 5.09 -> 0.00 mm, vias 1 -> 0
- net N$4: track 5.09 -> 2.54 mm, vias 1 -> 2
- net N$6: track 5.09 -> 2.54 mm
- net N$7: track 0.00 -> 2.54 mm, vias 0 -> 2
- added copper zone on layer 16, net N$7
- removed copper zone on layer 16, net N$5
Changed lines of the file:
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@@
 <grid distance="10" unitdist="mil" unit="mil" style="lines" multiple="1" display="no" altdistance="5" altunitdist="mil" altunit="mil"/>
 <layers>
-<layer number="1" name="Top" color="4" fill="1" visible="no" active="yes"/>
+<layer number="1" name="Top" color="4" fill="1" visible="yes" active="yes"/>
 <layer number="2" name="Route2" color="16" fill="1" visible="no" active="no"/>
 <layer number="3" name="Route3" color="17" fill="1" visible="no" active="no"/>
@@
 <layer number="14" name="Route14" color="22" fill="1" visible="no" active="no"/>
 <layer number="15" name="Route15" color="23" fill="1" visible="no" active="no"/>
-<layer number="16" name="Bottom" color="1" fill="1" visible="no" active="yes"/>
+<layer number="16" name="Bottom" color="1" fill="1" visible="yes" active="yes"/>
 <layer number="17" name="Pads" color="2" fill="1" visible="yes" active="yes"/>
 <layer number="18" name="Vias" color="2" fill="1" visible="yes" active="yes"/>
@@
 <layer number="22" name="bPlace" color="7" fill="1" visible="yes" active="yes"/>
 <layer number="23" name="tOrigins" color="15" fill="1" visible="yes" active="yes"/>
-<layer number="24" name="bOrigins" color="15" fill="1" visible="no" active="yes"/>
-<layer number="25" name="tNames" color="7" fill="1" visible="no" active="yes"/>
-<layer number="26" name="bNames" color="7" fill="1" visible="no" active="yes"/>
+<layer number="24" name="bOrigins" color="15" fill="1" visible="yes" active="yes"/>
+<layer number="25" name="tNames" color="7" fill="1" visible="yes" active="yes"/>
+<layer number="26" name="bNames" color="7" fill="1" visible="yes" active="yes"/>
 <layer number="27" name="tValues" color="7" fill="1" visible="yes" active="yes"/>
-<layer number="28" name="bValues" color="7" fill="1" visible="no" active="yes"/>
+<layer number="28" name="bValues" color="7" fill="1" visible="yes" active="yes"/>
 <layer number="29" name="tStop" color="7" fill="3" visible="yes" active="yes"/>
 <layer number="30" name="bStop" color="7" fill="6" visible="no" active="yes"/>
-<layer number="31" name="tCream" color="7" fill="4" visible="no" active="yes"/>
-<layer number="32" name="bCream" color="7" fill="5" visible="no" active="yes"/>
+<layer number="31" name="tCream" color="7" fill="4" visible="yes" active="yes"/>
+<layer number="32" name="bCream" color="7" fill="5" visible="yes" active="yes"/>
 <layer number="33" name="tFinish" color="6" fill="3" visible="no" active="yes"/>
 <layer number="34" name="bFinish" color="6" fill="6" visible="no" active="yes"/>
@@
 <hole x="6.0833" y="47.498" drill="3.429" locked="yes"/>
 <text x="33.655" y="10.795" size="1.778" layer="21">G</text>
-<text x="33.655" y="18.415" size="1.778" layer="21">R</text>
-<text x="33.655" y="25.4" size="1.778" layer="21">B</text>
+<text x="33.655" y="17.907" size="1.778" layer="21">R</text>
+<text x="33.655" y="24.892" size="1.778" layer="21">B</text>
 <text x="24.765" y="-3.81" size="1.778" layer="21">Benjamin Kittendorf</text>
 <text x="24.765" y="-6.35" size="1.778" layer="21">7/7/19</text>
@@
 <signals>
 <signal name="N$4">
-<contactref element="FETB" pad="3"/>
-<via x="21.59" y="25.4" extent="1-16" drill="1"/>
-<wire x1="22.8346" y1="23.368" x2="22.8346" y2="24.1554" width="1.27" layer="1"/>
-<wire x1="22.8346" y1="24.1554" x2="21.59" y2="25.4" width="1.27" layer="1"/>
-<polygon width="0.0762" layer="16">
-<vertex x="3.429" y="-0.254"/>
-<vertex x="14.351" y="-0.254"/>
-<vertex x="16.51" y="1.905"/>
-<vertex x="16.51" y="17.145"/>
-<vertex x="24.13" y="24.765"/>
-<vertex x="24.13" y="26.67"/>
-<vertex x="22.86" y="27.94"/>
-<vertex x="20.955" y="27.94"/>
-<vertex x="14.605" y="21.59"/>
-<vertex x="14.605" y="3.175"/>
-<vertex x="13.335" y="1.905"/>
-<vertex x="3.175" y="1.905"/>
-<vertex x="2.54" y="1.27"/>
-<vertex x="2.54" y="0.635"/>
-</polygon>
+<contactref element="FETB" pad="2"/>
 <contactref element="JP1" pad="2"/>
 <contactref element="JP1" pad="1"/>
 <wire x1="6.604" y1="0.889" x2="4.064" y2="0.889" width="1.905" layer="1"/>
-</signal>
-<signal name="N$5">
-<contactref element="FETR" pad="3"/>
-<via x="21.59" y="18.415" extent="1-16" drill="1"/>
-<wire x1="22.8346" y1="16.383" x2="22.8346" y2="17.1704" width="1.27" layer="1"/>
-<wire x1="22.8346" y1="17.1704" x2="21.59" y2="18.415" width="1.27" layer="1"/>
-<polygon width="0.0762" layer="16">
-<vertex x="15.24" y="-0.635"/>
-<vertex x="3.175" y="-0.635"/>
-<vertex x="2.54" y="-1.27"/>
-<vertex x="2.54" y="-1.905"/>
-<vertex x="3.429" y="-2.794"/>
-<vertex x="15.621" y="-2.794"/>
-<vertex x="19.685" y="1.27"/>
-<vertex x="19.685" y="12.7"/>
-<vertex x="24.13" y="17.145"/>
-<vertex x="24.13" y="19.685"/>
-<vertex x="22.86" y="20.955"/>
-<vertex x="20.955" y="20.955"/>
-<vertex x="17.145" y="17.145"/>
-<vertex x="17.145" y="1.27"/>
+<via x="34.29" y="23.368" extent="1-16" drill="1"/>
+<via x="34.29" y="28.194" extent="1-16" drill="1"/>
+<polygon width="0.1524" layer="16">
+<vertex x="3.556" y="2.286"/>
+<vertex x="2.794" y="1.524"/>
+<vertex x="2.794" y="0.254"/>
+<vertex x="3.302" y="-0.254"/>
+<vertex x="17.78" y="-0.254"/>
+<vertex x="24.13" y="6.096"/>
+<vertex x="24.13" y="15.748"/>
+<vertex x="30.48" y="22.098"/>
+<vertex x="34.798" y="22.098"/>
+<vertex x="35.306" y="22.606"/>
+<vertex x="35.306" y="28.702"/>
+<vertex x="34.798" y="29.21"/>
+<vertex x="29.718" y="29.21"/>
+<vertex x="20.574" y="20.066"/>
+<vertex x="20.574" y="5.842"/>
+<vertex x="17.018" y="2.286"/>
 </polygon>
-<contactref element="JP1" pad="4"/>
-<contactref element="JP1" pad="3"/>
-<wire x1="6.604" y1="-1.651" x2="4.064" y2="-1.651" width="1.905" layer="1"/>
+<wire x1="34.29" y1="23.368" x2="29.21" y2="25.654" width="0" layer="19" extent="1-1"/>
 </signal>
 <signal name="N$6">
-<contactref element="FETG" pad="3"/>
-<via x="21.59" y="11.43" extent="1-16" drill="1"/>
-<wire x1="22.8346" y1="9.398" x2="22.8346" y2="10.1854" width="1.27" layer="1"/>
-<wire x1="22.8346" y1="10.1854" x2="21.59" y2="11.43" width="1.27" layer="1"/>
-<polygon width="0.0762" layer="16">
-<vertex x="16.51" y="-3.175"/>
-<vertex x="3.175" y="-3.175"/>
-<vertex x="2.54" y="-3.81"/>
-<vertex x="2.54" y="-5.08"/>
-<vertex x="3.175" y="-5.715"/>
-<vertex x="18.415" y="-5.715"/>
-<vertex x="24.765" y="0.635"/>
-<vertex x="24.765" y="10.16"/>
-<vertex x="22.225" y="12.7"/>
-<vertex x="20.955" y="12.7"/>
-<vertex x="20.32" y="12.065"/>
-<vertex x="20.32" y="0.635"/>
-</polygon>
 <contactref element="JP1" pad="6"/>
 <contactref element="JP1" pad="5"/>
 <wire x1="6.604" y1="-4.191" x2="4.064" y2="-4.191" width="1.905" layer="1"/>
+<contactref element="FETG" pad="2"/>
+<via x="34.29" y="9.144" extent="1-16" drill="1"/>
+<polygon width="0.1524" layer="16">
+<vertex x="21.082" y="-3.048"/>
+<vertex x="3.302" y="-3.048"/>
+<vertex x="2.794" y="-3.556"/>
+<vertex x="2.794" y="-4.826"/>
+<vertex x="3.048" y="-5.08"/>
+<vertex x="22.098" y="-5.08"/>
+<vertex x="35.306" y="8.128"/>
+<vertex x="35.306" y="14.478"/>
+<vertex x="34.798" y="14.986"/>
+<vertex x="33.02" y="14.986"/>
+<vertex x="30.226" y="12.192"/>
+<vertex x="30.226" y="6.096"/>
+</polygon>
+<wire x1="34.29" y1="9.144" x2="29.21" y2="11.684" width="0" layer="19" extent="1-1"/>
 </signal>
 <signal name="5V">
@@
 <contactref element="U$1" pad="P24"/>
 <contactref element="U$1" pad="P40"/>
-<contactref element="FETG" pad="2"/>
-<contactref element="FETR" pad="2"/>
-<contactref element="FETB" pad="2"/>
 <contactref element="JP2" pad="3"/>
 <contactref element="R5" pad="1"/>
@@
 <vertex x="0" y="-8.89"/>
 </polygon>
-<polygon width="0.0762" layer="16">
+<contactref element="FETR" pad="3"/>
+<contactref element="FETB" pad="3"/>
+<contactref element="FETG" pad="3"/>
+<polygon width="0.1524" layer="16">
 <vertex x="0" y="53.34"/>
 <vertex x="48.26" y="53.34"/>
-<vertex x="48.26" y="-8.89"/>
-<vertex x="24.13" y="-8.89"/>
-<vertex x="21.59" y="-6.35"/>
-<vertex x="21.59" y="-3.81"/>
-<vertex x="25.4" y="0"/>
-<vertex x="25.4" y="10.795"/>
-<vertex x="22.86" y="13.335"/>
-<vertex x="22.86" y="14.605"/>
-<vertex x="24.765" y="16.51"/>
-<vertex x="24.765" y="27.94"/>
-<vertex x="24.13" y="28.575"/>
-<vertex x="20.32" y="28.575"/>
-<vertex x="13.97" y="22.225"/>
-<vertex x="13.97" y="3.81"/>
-<vertex x="12.7" y="2.54"/>
-<vertex x="0" y="2.54"/>
+<vertex x="48.26" y="-8.636"/>
+<vertex x="48.514" y="-8.89"/>
+<vertex x="25.654" y="-8.89"/>
+<vertex x="24.638" y="-7.874"/>
+<vertex x="24.638" y="-4.318"/>
+<vertex x="30.48" y="1.524"/>
+<vertex x="33.274" y="1.524"/>
+<vertex x="37.592" y="5.842"/>
+<vertex x="37.592" y="28.702"/>
+<vertex x="36.576" y="29.718"/>
+<vertex x="29.464" y="29.718"/>
+<vertex x="20.066" y="20.32"/>
+<vertex x="20.066" y="6.096"/>
+<vertex x="16.764" y="2.794"/>
+<vertex x="3.302" y="2.794"/>
+<vertex x="0" y="6.096"/>
 </polygon>
 </signal>
@@
 <via x="34.29" y="30.48" extent="1-16" drill="0.35"/>
 </signal>
+<signal name="N$7">
+<contactref element="JP1" pad="4"/>
+<contactref element="JP1" pad="3"/>
+<wire x1="6.604" y1="-1.651" x2="4.064" y2="-1.651" width="1.905" layer="1"/>
+<contactref element="FETR" pad="2"/>
+<via x="34.29" y="16.256" extent="1-16" drill="1"/>
+<via x="34.29" y="20.828" extent="1-16" drill="1"/>
+<polygon width="0.1524" layer="16">
+<vertex x="3.302" y="-0.508"/>
+<vertex x="2.794" y="-1.016"/>
+<vertex x="2.794" y="-2.286"/>
+<vertex x="3.048" y="-2.54"/>
+<vertex x="20.828" y="-2.54"/>
+<vertex x="29.718" y="6.35"/>
+<vertex x="29.718" y="12.192"/>
+<vertex x="32.766" y="15.24"/>
+<vertex x="34.798" y="15.24"/>
+<vertex x="35.306" y="15.748"/>
+<vertex x="35.306" y="21.336"/>
+<vertex x="34.798" y="21.844"/>
+<vertex x="30.734" y="21.844"/>
+<vertex x="24.638" y="15.748"/>
+<vertex x="24.638" y="6.096"/>
+<vertex x="18.034" y="-0.508"/>
+</polygon>
+<wire x1="34.29" y1="20.828" x2="29.21" y2="18.669" width="0" layer="19" extent="1-1"/>
+</signal>
+<signal name="N6">
+<via x="34.29" y="13.97" extent="1-16" drill="1"/>
+</signal>
 </signals>
